File: Solar Cell offgrid Power.kicad_pcb (KiCad board)
At the start: 2 copper layers, 124.5 x 68.1 mm, 13 parts, among them J1 Conn_01x10_Socket, J2 Conn_01x10_Pin, J3 Screw_Terminal_01x02, J4 Conn_02x03_Counter_Clockwise, Q1 S8550

Commit message: Add files via upload
Parts:
- moved Q1 1.46 mm to (129.0, 88.8)
Connections:
- Q1 pad 1: Net-(D1-K) -> Net-(Q1-B)
- Q1 pad 2: Net-(Q1-B) -> Net-(D1-K)
Routing:
- net Net-(D1-K): track 15.7 -> 20.1 mm
- net PWR: track 181.2 -> 182.7 mm

Commit message: Add files via upload
Parts:
- added BT1: BK-18650-PC2, Battery:batery holder BAT_BK-18650-PC2, F.Cu at (172.8, 77.3)
- added G***: LOGO, AeonLabs Logos:smart build design, F.Cu at (166.1, 123.5)
- added REF**: OSHW-Logo2_14.6x12mm_SilkScreen, Symbol:OSHW-Logo2_14.6x12mm_SilkScreen, F.Cu at (188.6, 124.2)
- moved J4 19.7 mm to (124.4, 131.9), turned to 0 degrees
Connections:
- net Net-(D1-K) renamed BAT+
Routing:
- net BAT+: track 20.1 -> 25.6 mm
- net GND: track 277.3 -> 282.0 mm
Other:
- board text added: "BAT GND"
- board text added: "BAT+"
- board text added: "CELL +"
- board text added: "CELL GND"
- board text added: "CONNECT TO OTHER SOLAR TILE"
- board text added: "MAIN POWER"

Commit message: Add files via upload
Parts:
- added BK1: Copper Track Breaker, AeonLabs_Connectors:Copper Track Breaker 2 points, F.Cu at (175.0, 111.9)
- added BK2: Copper Track Breaker, AeonLabs_Connectors:Copper Track Breaker 2 points, F.Cu at (178.1, 111.9)
- added BK3: Copper Track Breaker, AeonLabs_Connectors:Copper Track Breaker 2 points, F.Cu at (181.1, 111.9)
- added BK4: Copper Track Breaker, AeonLabs_Connectors:Copper Track Breaker 2 points, F.Cu at (160.6, 112.0)
- added BK5: Copper Track Breaker, AeonLabs_Connectors:Copper Track Breaker 2 points, F.Cu at (163.3, 112.0)
- added BK6: Copper Track Breaker, AeonLabs_Connectors:Copper Track Breaker 2 points, F.Cu at (166.0, 112.0)
- added BK7: Copper Track Breaker, AeonLabs_Connectors:Copper Track Breaker 2 points, F.Cu at (168.9, 111.9)
- added BK8: Copper Track Breaker, AeonLabs_Connectors:Copper Track Breaker 2 points, F.Cu at (172.0, 111.9)
- moved G*** 43.8 mm to (122.6, 129.1)
- moved REF** 28.9 mm to (217.5, 123.0)
- moved R1 11.4 mm to (128.0, 93.4)
- moved Q1 7.20 mm to (121.8, 88.4)
- moved D1 6.24 mm to (128.1, 89.6)
- moved BT1 0.90 mm to (172.1, 78.0)
- moved J4 0.35 mm to (124.3, 132.2)
- moved BAT_POS1 0.23 mm to (131.2, 77.2)
Connections:
- J1 pad 1: unconnected-(J1-Pin_1-Pad1) -> Conn_track_1
- J1 pad 10: unconnected-(J1-Pin_10-Pad10) -> Conn_track_10
- J1 pad 2: unconnected-(J1-Pin_2-Pad2) -> Conn_track_2
- J1 pad 3: unconnected-(J1-Pin_3-Pad3) -> Conn_track_3
- J1 pad 4: PWR -> Conn_track_4
- J1 pad 7: GND -> Conn_track_7
- J1 pad 8: unconnected-(J1-Pin_8-Pad8) -> Conn_track_8
- J1 pad 9: unconnected-(J1-Pin_9-Pad9) -> Conn_track_9
- J2 pad 1: unconnected-(J2-Pin_1-Pad1) -> Conn_track_1
- J2 pad 10: unconnected-(J2-Pin_10-Pad10) -> Conn_track_10
- J2 pad 2: unconnected-(J2-Pin_2-Pad2) -> Conn_track_2
- J2 pad 3: unconnected-(J2-Pin_3-Pad3) -> Conn_track_3
- J2 pad 4: PWR -> Conn_track_4
- J2 pad 7: GND -> Conn_track_7
- J2 pad 8: unconnected-(J2-Pin_8-Pad8) -> Conn_track_8
- J2 pad 9: unconnected-(J2-Pin_9-Pad9) -> Conn_track_9
Routing:
- net Conn_track_10: track 0.00 -> 135.1 mm, vias 0 -> 1
- net Conn_track_9: track 0.00 -> 131.9 mm, vias 0 -> 1
- net Conn_track_8: track 0.00 -> 131.1 mm, vias 0 -> 1
- net Conn_track_7: track 0.00 -> 131.0 mm, vias 0 -> 1
- net Conn_track_4: track 0.00 -> 118.8 mm, vias 0 -> 1
- net Conn_track_3: track 0.00 -> 116.3 mm, vias 0 -> 1
- net Conn_track_2: track 0.00 -> 115.6 mm, vias 0 -> 1
- net Conn_track_1: track 0.00 -> 115.4 mm, vias 0 -> 1
- net BAT+: track 25.6 -> 134.3 mm, vias 0 -> 2
- net PWR: track 182.7 -> 196.6 mm
- net Net-(D1-A): track 111.4 -> 117.1 mm
- net GND: track 282.0 -> 276.9 mm
- net Net-(J4-Pin_1): track 9.16 -> 5.64 mm
- net Net-(Q1-B): track 18.2 -> 14.9 mm
Other:
- board text added: "1"
- board text added: "10"
- board text added: "2"
- board text added: "3"
- board text added: "4"
- board text added: "7"
- board text added: "8"
- board text added: "9"
- board text added: "Battery Channel IO"
- board text added: "FOR SINGLE BLUE SOLAR TILE 2x 18650 liPo BATTERY"
- board text added: "make sure you have a unique channel number on the rail"
