File: Solar Cell offgrid Power.kicad_sch (KiCad schematic)
At the start: 11 parts, among them J1 Conn_01x10_Socket, J2 Conn_01x10_Pin, J3 Screw_Terminal_01x02, J4 Conn_02x03_Counter_Clockwise, Q1 S8550

Commit message: Add files via upload
Connections:
- net at BAT_POS1.1, D1.1 (K): now also Q1.2 (E); no longer Q1.1 (E)
- net at R1.2: now also Q1.1 (B); no longer Q1.2 (B)
Other:
- moved on the sheet: R1
Changed lines of the file:
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@@
 (kicad_sch (version 20230121) (generator eeschema)
   (paper "A4")
+  (junction (at 132.5626 65.3542) (diameter 0) (color 0 0 0 0)
+  )
   (junction (at 144.1196 65.3542) (diameter 0) (color 0 0 0 0)
   )
-  (junction (at 132.461 65.3796) (diameter 0) (color 0 0 0 0)
+  (wire (pts (xy 132.5626 65.3542) (xy 132.5626 74.2188))
+    (stroke (width 0) (type default))
   )
   (wire (pts (xy 144.1196 65.3542) (xy 145.7198 65.3542))
     (stroke (width 0) (type default))
   )
-  (wire (pts (xy 132.461 82.3976) (xy 132.461 80.4418))
-    (stroke (width 0) (type default))
-  )
-  (wire (pts (xy 134.7978 65.3542) (xy 132.461 65.3542))
-    (stroke (width 0) (type default))
-  )
-  (wire (pts (xy 144.1196 72.39) (xy 148.0312 72.39))
+  (wire (pts (xy 132.5626 86.3346) (xy 132.5626 84.3788))
+    (stroke (width 0) (type default))
+  )
+  (wire (pts (xy 134.7978 65.3542) (xy 132.5626 65.3542))
+    (stroke (width 0) (type default))
+  )
+  (wire (pts (xy 144.1196 72.39) (xy 148.209 72.39))
     (stroke (width 0) (type default))
   )
@@
     (stroke (width 0) (type default))
   )
-  (wire (pts (xy 148.0312 72.39) (xy 148.0312 75.3364))
-    (stroke (width 0) (type default))
-  )
-  (wire (pts (xy 132.461 65.3796) (xy 132.461 70.2818))
+  (wire (pts (xy 148.209 72.39) (xy 148.209 79.2988))
     (stroke (width 0) (type default))
   )
@@
     (stroke (width 0) (type default))
   )
-  (wire (pts (xy 140.3858 75.3364) (xy 140.3858 75.3618))
+  (wire (pts (xy 132.5626 65.3542) (xy 132.461 65.3542))
     (stroke (width 0) (type default))
   )
@@
     (stroke (width 0) (type default))
   )
-  (wire (pts (xy 140.3858 75.3618) (xy 140.081 75.3618))
-    (stroke (width 0) (type default))
-  )
   (wire (pts (xy 142.4178 65.3542) (xy 144.1196 65.3542))
     (stroke (width 0) (type default))
@@
     (stroke (width 0) (type default))
   )
-  (wire (pts (xy 140.4112 75.3364) (xy 140.3858 75.3364))
+  (wire (pts (xy 140.1826 79.2988) (xy 140.589 79.2988))
     (stroke (width 0) (type default))
   )
@@
     )
   )
-  (global_label "PWR" (shape input) (at 132.461 82.3976 0) (fields_autoplaced)
-    (effects (font (size 1.27 1.27)) (justify left))
-    (property "Intersheetrefs" "${INTERSHEET_REFS}" (at 139.3582 82.3976 0)
+  (global_label "PWR" (shape input) (at 132.5626 86.3346 0) (fields_autoplaced)
+    (effects (font (size 1.27 1.27)) (justify left))
+    (property "Intersheetrefs" "${INTERSHEET_REFS}" (at 139.4598 86.3346 0)
       (effects (font (size 1.27 1.27)) (justify left) hide)
     )
@@
     )
   )
-  (symbol (lib_id "power:GND") (at 149.4028 65.3542 0) (unit 1)
-    (in_bom yes) (on_board yes) (dnp no) (fields_autoplaced)
-    (property "Reference" "#PWR01" (at 149.4028 71.7042 0)
-      (effects (font (size 1.27 1.27)) hide)
-    )
-    (property "Value" "GND" (at 149.4028 70.5104 0)
-      (effects (font (size 1.27 1.27)))
-    )
-    (property "Footprint" "" (at 149.4028 65.3542 0)
-      (effects (font (size 1.27 1.27)) hide)
-    )
-    (property "Datasheet" "" (at 149.4028 65.3542 0)
-      (effects (font (size 1.27 1.27)) hide)
-    )
-    (pin "1")
-    (instances
-      (project "Solar Cell offgrid Power"
-        (path "/36c3529d-7964-4040-afe2-98add62a25cb"
-          (reference "#PWR01") (unit 1)
-        )
-      )
-    )
-  )
-  (symbol (lib_id "power:GND") (at 115.57 65.5066 0) (unit 1)
-    (in_bom yes) (on_board yes) (dnp no) (fields_autoplaced)
-    (property "Reference" "#PWR02" (at 115.57 71.8566 0)
-      (effects (font (size 1.27 1.27)) hide)
-    )
-    (property "Value" "GND" (at 115.57 70.6628 0)
-      (effects (font (size 1.27 1.27)))
-    )
-    (property "Footprint" "" (at 115.57 65.5066 0)
-      (effects (font (size 1.27 1.27)) hide)
-    )
-    (property "Datasheet" "" (at 115.57 65.5066 0)
-      (effects (font (size 1.27 1.27)) hide)
-    )
-    (pin "1")
-    (instances
-      (project "Solar Cell offgrid Power"
-        (path "/36c3529d-7964-4040-afe2-98add62a25cb"
-          (reference "#PWR02") (unit 1)
-        )
-      )
-    )
-  )
-  (symbol (lib_id "Transistor_BJT:S8550") (at 135.001 75.3618 180) (unit 1)
-    (in_bom yes) (on_board yes) (dnp no) (fields_autoplaced)
-    (property "Reference" "Q1" (at 129.5908 75.9968 0)
-      (effects (font (size 1.27 1.27)) (justify left))
-    )
-    (property "Value" "S8550" (at 129.5908 73.4568 0)
-      (effects (font (size 1.27 1.27)) (justify left))
-    )
-    (property "Footprint" "Package_TO_SOT_SMD:SOT-23-3" (at 129.921 73.4568 0)
+  (symbol (lib_id "Transistor_BJT:S8550") (at 135.1026 79.2988 180) (unit 1)
+    (in_bom yes) (on_board yes) (dnp no) (fields_autoplaced)
+    (property "Reference" "Q1" (at 129.4892 78.6638 0)
+      (effects (font (size 1.27 1.27)) (justify left))
+    )
+    (property "Value" "S8550" (at 129.4892 81.2038 0)
+      (effects (font (size 1.27 1.27)) (justify left))
+    )
+    (property "Footprint" "Package_TO_SOT_SMD:SOT-23-3" (at 146.6342 92.6592 0)
       (effects (font (size 1.27 1.27) italic) (justify left) hide)
     )
-    (property "Datasheet" "http://www.unisonic.com.tw/datasheet/S8550.pdf" (at 135.001 75.3618 0)
+    (property "Datasheet" "http://www.unisonic.com.tw/datasheet/S8550.pdf" (at 149.225 94.5388 0)
       (effects (font (size 1.27 1.27)) (justify left) hide)
     )
@@
         (path "/36c3529d-7964-4040-afe2-98add62a25cb"
           (reference "Q1") (unit 1)
+        )
+      )
+    )
+  )
+  (symbol (lib_id "power:GND") (at 149.4028 65.3542 0) (unit 1)
+    (in_bom yes) (on_board yes) (dnp no) (fields_autoplaced)
+    (property "Reference" "#PWR01" (at 149.4028 71.7042 0)
+      (effects (font (size 1.27 1.27)) hide)
+    )
+    (property "Value" "GND" (at 149.4028 70.5104 0)
+      (effects (font (size 1.27 1.27)))
+    )
+    (property "Footprint" "" (at 149.4028 65.3542 0)
+      (effects (font (size 1.27 1.27)) hide)
+    )
+    (property "Datasheet" "" (at 149.4028 65.3542 0)
+      (effects (font (size 1.27 1.27)) hide)
+    )
+    (pin "1")
+    (instances
+      (project "Solar Cell offgrid Power"
+        (path "/36c3529d-7964-4040-afe2-98add62a25cb"
+          (reference "#PWR01") (unit 1)
+        )
+      )
+    )
+  )
+  (symbol (lib_id "power:GND") (at 115.57 65.5066 0) (unit 1)
+    (in_bom yes) (on_board yes) (dnp no) (fields_autoplaced)
+    (property "Reference" "#PWR02" (at 115.57 71.8566 0)
+      (effects (font (size 1.27 1.27)) hide)
+    )
+    (property "Value" "GND" (at 115.57 70.6628 0)
+      (effects (font (size 1.27 1.27)))
+    )
+    (property "Footprint" "" (at 115.57 65.5066 0)
+      (effects (font (size 1.27 1.27)) hide)
+    )
+    (property "Datasheet" "" (at 115.57 65.5066 0)
+      (effects (font (size 1.27 1.27)) hide)
+    )
+    (pin "1")
+    (instances
+      (project "Solar Cell offgrid Power"
+        (path "/36c3529d-7964-4040-afe2-98add62a25cb"
+          (reference "#PWR02") (unit 1)
         )
       )
@@
     )
   )
-  (symbol (lib_id "Device:R") (at 144.2212 75.3364 270) (unit 1)
+  (symbol (lib_id "Device:R") (at 144.399 79.2988 270) (unit 1)
     (in_bom yes) (on_board yes) (dnp no)
-    (property "Reference" "R1" (at 144.6784 77.5462 90)
-      (effects (font (size 1.27 1.27)))
-    )
-    (property "Value" "5K6" (at 144.2974 75.4888 90)
-      (effects (font (size 1.27 1.27)))
-    )
-    (property "Footprint" "Resistor_SMD:R_1210_3225Metric" (at 144.2212 73.5584 90)
-      (effects (font (size 1.27 1.27)) hide)
-    )
-    (property "Datasheet" "~" (at 144.2212 75.3364 0)
-      (effects (font (size 1.27 1.27)) hide)
-    )
+    (property "Reference" "R1" (at 144.8562 81.5086 90)
+      (effects (font (size 1.27 1.27)))
+    )
+    (property "Value" "5K6" (at 144.4752 79.4512 90)
+      (effects (font (size 1.27 1.27)))
+    )
+    (property "Footprint" "Resistor_SMD:R_1210_3225Metric" (at 144.399 77.5208 90)
+      (effects (font (size 1.27 1.27)) hide)
+    )
+    (property "Datasheet" "~" (at 144.399 79.2988 0)
+      (effects (font (size 1.27 1.27)) hide)
+    )

Commit message: Add files via upload
Parts:
- added BT1: BK-18650-PC2, Battery:batery holder BAT_BK-18650-PC2, symbol Battery_Management:BK-18650-PC2
Connections:
- net GND: now also BT1.-
- net BAT+: now reaches BAT_POS1.1, D1.1 (K), Q1.2 (E)
- net BAT+: now also BT1.+
Changed lines of the file:
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@@
+    )
+  )
+  (global_label "BAT+" (shape input) (at 122.7328 44.1452 180) (fields_autoplaced)
+    (effects (font (size 1.27 1.27)) (justify right))
+    (property "Intersheetrefs" "${INTERSHEET_REFS}" (at 114.9284 44.1452 0)
+      (effects (font (size 1.27 1.27)) (justify right) hide)
     )
   )
@@
     (effects (font (size 1.27 1.27)) (justify left))
     (property "Intersheetrefs" "${INTERSHEET_REFS}" (at 139.4598 86.3346 0)
+      (effects (font (size 1.27 1.27)) (justify left) hide)
+    )
+  )
+  (global_label "BAT+" (shape input) (at 127 65.3796 90) (fields_autoplaced)
+    (effects (font (size 1.27 1.27)) (justify left))
+    (property "Intersheetrefs" "${INTERSHEET_REFS}" (at 127 57.5752 90)
       (effects (font (size 1.27 1.27)) (justify left) hide)
     )
@@
     )
   )
+  (symbol (lib_id "Battery_Management:BK-18650-PC2") (at 130.3528 44.1452 0) (unit 1)
+    (in_bom yes) (on_board yes) (dnp no) (fields_autoplaced)
+    (property "Reference" "BT1" (at 129.7178 38.1 0)
+      (effects (font (size 1.27 1.27)))
+    )
+    (property "Value" "BK-18650-PC2" (at 129.7178 40.64 0)
+      (effects (font (size 1.27 1.27)))
+    )
+    (property "Footprint" "Battery:batery holder BAT_BK-18650-PC2" (at 130.4544 36.6268 0)
+      (effects (font (size 1.27 1.27)) (justify bottom) hide)
+    )
+    (property "Datasheet" "" (at 130.3528 44.1452 0)
+      (effects (font (size 1.27 1.27)) hide)
+    )
+    (property "MANUFACTURER" "MPD" (at 130.3528 44.1452 0)
+      (effects (font (size 1.27 1.27)) (justify bottom) hide)
+    )
+    (property "STANDARD" "Manufacturer Recommendations" (at 130.2512 32.7152 0)
+      (effects (font (size 1.27 1.27)) (justify bottom) hide)
+    )
+    (property "PARTREV" "F" (at 130.3528 44.1452 0)
+      (effects (font (size 1.27 1.27)) (justify bottom) hide)
+    )
+    (property "MAXIMUM_PACKAGE_HEIGHT" "21.41 mm" (at 129.3876 29.1084 0)
+      (effects (font (size 1.27 1.27)) (justify bottom) hide)
+    )
+    (pin "+")
+    (pin "-")
+    (instances
+      (project "Solar Cell offgrid Power"
+        (path "/36c3529d-7964-4040-afe2-98add62a25cb"
+          (reference "BT1") (unit 1)
+        )
+      )
+    )
+  )
   (symbol (lib_id "Connector_Generic:Conn_02x03_Counter_Clockwise") (at 95.8596 137.5156 0) (unit 1)
     (in_bom yes) (on_board yes) (dnp no) (fields_autoplaced)
@@
         )
       )
+    )
+  )
+  (symbol (lib_id "power:GND") (at 137.9728 44.1452 0) (unit 1)
+    (in_bom yes) (on_board yes) (dnp no) (fields_autoplaced)
+    (property "Reference" "#PWR03" (at 137.9728 50.4952 0)
+      (effects (font (size 1.27 1.27)) hide)
+    )
+    (property "Value" "GND" (at 137.9728 49.3014 0)
+      (effects (font (size 1.27 1.27)))
+    )
+    (property "Footprint" "" (at 137.9728 44.1452 0)
+      (effects (font (size 1.27 1.27)) hide)
+    )
+    (property "Datasheet" "" (at 137.9728 44.1452 0)
+      (effects (font (size 1.27 1.27)) hide)
+    )
+    (pin "1")
+    (instances
+      (project "Solar Cell offgrid Power"
+        (path "/36c3529d-7964-4040-afe2-98add62a25cb"
+          (reference "#PWR03") (unit 1)
+        )
+      )

Commit message: Add files via upload
Parts:
- added BK1, BK2, BK3, BK4, BK5, BK6, BK7, BK8: Copper Track Breaker, AeonLabs_Connectors:Copper Track Breaker 2 points, symbol AeonLabs_Connectors:Copper_Track_Break_2_points
Connections:
- net BAT+: now also BK1.1, BK2.1, BK3.1, BK4.1, BK5.1, BK6.1, BK7.1, BK8.1
- net GND: no longer J1.7 (Pin_7), J2.7 (Pin_7)
- net PWR: no longer J1.4 (Pin_4), J2.4 (Pin_4)
- net Conn_track_1: now reaches J2.1 (Pin_1)
- net Conn_track_1: now also J1.1 (Pin_1), BK4.2
- net Conn_track_10: now reaches J2.10 (Pin_10)
- net Conn_track_10: now also J1.10 (Pin_10), BK3.2
- net Conn_track_2: now reaches J2.2 (Pin_2)
- net Conn_track_2: now also J1.2 (Pin_2), BK5.2
- net Conn_track_3: now reaches J2.3 (Pin_3)
- net Conn_track_3: now also J1.3 (Pin_3), BK6.2
- net Conn_track_8: now reaches J2.8 (Pin_8)
- net Conn_track_8: now also J1.8 (Pin_8), BK1.2
- net Conn_track_9: now reaches J2.9 (Pin_9)
- net Conn_track_9: now also J1.9 (Pin_9), BK2.2
- new net Conn_track_4: BK7.2, J1.4 (Pin_4), J2.4 (Pin_4)
- new net Conn_track_7: BK8.2, J1.7 (Pin_7), J2.7 (Pin_7)
Other:
- moved on the sheet: J2
